File: Zynq-Carrier-Template.kicad_pcb (KiCad board)
At the start: 2 copper layers, 49 x 41 mm, 7 parts, among them J1 Zynq_SoM, J3 USB_C_Receptacle_USB2.0_16P, U1 BQ25629RYKR

Commit message: Import 1uH Inductor
Parts:
- added REF**: IND_P3519R_API, 1uH_Inductor:IND_P3519R_API, F.Cu at (135.2, 107.6)
